File: Vegapod 24-25/Sense & Control/Foundation Schematic/Foundation VCU.kicad_sch (KiCad schematic)
At the start: 53 parts, among them J4 615008137421, J5 Conn_01x04_Pin, J7 Conn_01x03_Pin, P1 USB_C_Plug_USB2.0, SW1 SW_rst, U1 STM32G474RETx, U2 ADM3050EBRIZ, U3 USBLC6-2SC6, U4 AMS1117-3.3, Y1 Crystal

Commit message: Add files via upload
Parts:
- added D8: BLUE LED, LED_SMD:LED_0805_2012Metric_Pad1.15x1.40mm_HandSolder, symbol Device:LED
- added J1: Conn_01x02_Pin, Connector_PinHeader_2.54mm:PinHeader_1x02_P2.54mm_Vertical, symbol Connector:Conn_01x02_Pin
- added J2: Conn_01x04_Pin, Connector_PinHeader_2.54mm:PinHeader_1x04_P2.54mm_Vertical, symbol Connector:Conn_01x04_Pin
- added R16: 220, Resistor_SMD:R_0805_2012Metric_Pad1.20x1.40mm_HandSolder, symbol Device:R
- added R17: 10K, Resistor_SMD:R_0805_2012Metric_Pad1.20x1.40mm_HandSolder, symbol Device:R
- added SW2: SW_rst, Button_Switch_SMD:SW_SPST_FSMSM, symbol Switch:SW_Push
- added U5: HC-05, HC-05:XCVR_HC-05, symbol HC-05:HC-05
Connections:
- net +3.3V: now also SW2.2, U5.12 (3.3_VCC)
- net +5V: now also J4.3; no longer J4.6
- net CAN_H: now also J4.1; no longer J4.3
- net GND: now also J4.8, J4.S1, J4.S2, D8.1 (K), R17.1, U5.13 (GND), U5.21 (GND), U5.22 (GND); no longer J4.7
- net LD6: now also U1.41 (PC9)
- net MVCU_HB: now also J4.7; no longer J4.S1, J4.S2
- net USART1_RX: now also J4.5; no longer J4.1
- net USART1_TX: now also J4.4; no longer J4.5
- net VCU_HB: now also J4.6; no longer J4.8
- net BT_UART_Rx: now reaches U1.14 (PA2)
- net BT_UART_Rx: now also J1.2 (Pin_2), U5.1 (UART-TX)
- net BT_UART_Tx: now reaches U1.17 (PA3)
- net BT_UART_Tx: now also J1.1 (Pin_1), U5.2 (UART-RX)
- new net: D8.2 (A), R16.1
- new net: R17.2, SW2.1, U5.34 (PIO[11])
- new net: J2.1 (Pin_1), U5.17 (SPI_MOSI)
- new net: J2.2 (Pin_2), U5.16 (~{SPI_CSB})
- new net: J2.3 (Pin_3), U5.19 (SPI_CLK)
- new net: J2.4 (Pin_4), U5.18 (SPI_MISO)
- new net: R16.2, U5.31 (PIO[8])
- no-connect marks 3 -> 23
Other:
- note added: "BT Programming"
- note removed: "sw_boot0"
- moved on the sheet: R10
